File: HW2/New_Project/schematics.brd (EAGLE design)
At the start: 160 x 100 mm, 24 parts, among them J1 USB-MB-H

Commit message: final update
Parts:
- moved J2 107.2 mm to (74.9, 41.9), turned to 90 degrees
- moved J1 100.8 mm to (3.81, 92.7)
- moved U$1 96.0 mm to (53.3, 49.5)
Connections:
- removed net A4: J2.6, U$1.34
- removed net B4: J2.5, U$1.33
- removed net LED: LED2.A
- removed net USER: R4.1, U$5.1
- new net A4/LED: J2.6, LED2.A, U$1.34
- new net B4/USER: J2.5, R4.1, U$1.33, U$5.1
Other:
- board size 160 x 100 mm -> 100 x 100 mm
