File: HW3/New_Project/schematics.brd (EAGLE design)
At the start: 100 x 100 mm, 24 parts, among them J1 USB-MB-H

Commit message: initial
Routing:
- net GND: track 0.00 -> 27.0 mm
Changed lines of the file:
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@@
 <vertex x="1.27" y="1.27"/>
 </polygon>
-<wire x1="62.738" y1="51.689" x2="59.14" y2="50.33" width="0" layer="19" extent="1-1"/>
-<wire x1="53.34" y1="55.33" x2="55.88" y2="58.42" width="0" layer="19" extent="1-1"/>
-<wire x1="47.54" y1="49.53" x2="43.688" y2="51.689" width="0" layer="19" extent="1-1"/>
-<wire x1="52.54" y1="43.73" x2="48.26" y2="39.37" width="0" layer="19" extent="1-1"/>
+<wire x1="59.14" y1="50.33" x2="60.76673125" y2="50.33" width="0.4064" layer="1"/>
+<wire x1="60.76673125" y1="50.33" x2="61.1886" y2="49.90813125" width="0.4064" layer="1"/>
+<wire x1="61.1886" y1="49.90813125" x2="61.1886" y2="48.739425" width="0.4064" layer="1"/>
+<wire x1="61.1886" y1="48.739425" x2="62.201425" y2="47.7266" width="0.4064" layer="1"/>
+<wire x1="62.201425" y1="47.7266" x2="63.274575" y2="47.7266" width="0.4064" layer="1"/>
+<wire x1="63.274575" y1="47.7266" x2="64.1604" y2="48.612425" width="0.4064" layer="1"/>
+<wire x1="64.1604" y1="48.612425" x2="64.1604" y2="49.812575" width="0.4064" layer="1"/>
+<wire x1="62.738" y1="51.234975" x2="62.738" y2="51.689" width="0.4064" layer="1"/>
+<wire x1="64.1604" y1="49.812575" x2="62.738" y2="51.234975" width="0.4064" layer="1"/>
+<wire x1="43.688" y1="51.689" x2="45.847" y2="49.53" width="0.4064" layer="1"/>
+<wire x1="45.847" y1="49.53" x2="47.54" y2="49.53" width="0.4064" layer="1"/>
+<wire x1="55.88" y1="58.42" x2="55.72710625" y2="58.42" width="0.4064" layer="1"/>
+<wire x1="55.72710625" y1="58.42" x2="53.34" y2="56.03289375" width="0.4064" layer="1"/>
+<wire x1="53.34" y1="56.03289375" x2="53.34" y2="55.33" width="0.4064" layer="1"/>
+<wire x1="48.26" y1="39.45" x2="48.26" y2="39.37" width="0.4064" layer="1"/>
+<wire x1="52.54" y1="43.73" x2="52.3456" y2="43.5356" width="0.4064" layer="1"/>
+<wire x1="51.79346875" y1="41.2242" x2="50.0342" y2="41.2242" width="0.4064" layer="1"/>
+<wire x1="50.0342" y1="41.2242" x2="48.26" y2="39.45" width="0.4064" layer="1"/>
+<wire x1="52.3456" y1="43.5356" x2="52.3456" y2="41.77633125" width="0.4064" layer="1"/>
+<wire x1="52.3456" y1="41.77633125" x2="51.79346875" y2="41.2242" width="0.4064" layer="1"/>
 </signal>
 <signal name="N$2">
@@
 <mfgpreviewcolor name="substratecolor" color="0xFF786E46"/>
 </mfgpreviewcolors>
+<errors>
+</errors>
 </board>
 </drawing>
